Commit message: Fixed urdf Fixed urdf to work in ROS2 Create sample launch file that loads the model in RVIZ

File: urdf/gazebo.xacro (robot description, xacro)
@@ -1,18 +1,18 @@
 <?xml version="1.0"?>
 <robot>
-    <gazebo>
-        <plugin name="gazebo_ros_control" filename="libgazebo_ros_control.so">
-            <robotNamespace>/z1_gazebo</robotNamespace>
-            <robotSimType>gazebo_ros_control/DefaultRobotHWSim</robotSimType>
-        </plugin>
-    </gazebo>
-    <gazebo reference="link04">
-        <self_collide>true</self_collide>
-    </gazebo>
-    <gazebo reference="link05">
-        <self_collide>true</self_collide>
-    </gazebo>
-    <gazebo reference="link06">
-        <self_collide>true</self_collide>
-    </gazebo>
+<gazebo>
+<plugin name="gazebo_ros_control" filename="libgazebo_ros_control.so">
+<robotNamespace>/z1_gazebo</robotNamespace>
+<robotSimType>gazebo_ros_control/DefaultRobotHWSim</robotSimType>
+</plugin>
+</gazebo>
+<gazebo reference="link04">
+<self_collide>true</self_collide>
+</gazebo>
+<gazebo reference="link05">
+<self_collide>true</self_collide>
+</gazebo>
+<gazebo reference="link06">
+<self_collide>true</self_collide>
+</gazebo>
 </robot>

File: urdf/z1.ros2_control.xacro (robot description, xacro)
@@ -1,3 +1,3 @@
-<?xl version="1.0"?>
+<?xml version="1.0"?>
 <!-- This file is based on ur.ros2_contro.xacro provided by Universal Robots for     -->
 <!-- their robots, but with data ported for the Z1 manipulator from alientree.       -->
@@ -7,5 +7,5 @@
   <xacro:macro name="z1_ros2_control" params="
     name
-    sim_ignition:=false
+    sim_ignition:=true
     prefix
     ">
@@ -16,10 +16,10 @@
         </xacro:if>
         <xacro:unless value="${sim_ignition}">
-          <plugin> unitree_z1_hw_interface/z1_effort_hw_interface</plugin>
+          <plugin>unitree_z1_hw_interface/UnitreeZ1HWInterface</plugin>
           <param name="gripper">true</param>
           <!-- add other necessary parameters here -->
         </xacro:unless>
       </hardware>
-      <joint name="${prefix}shoulder_pan_joint">
+      <joint name="$(arg prefix)shoulder_pan_joint">
         <command_interface name="position">
           <param name="min"> ${joint1_PositionMin} </param>
@@ -38,5 +38,5 @@
         <state_interface name="effort"/>
       </joint>
-      <joint name="${prefix}shoulder_lift_joint">
+      <joint name="$(arg prefix)shoulder_lift_joint">
         <command_interface name="position">
           <param name="min"> ${joint1_PositionMin} </param>
@@ -55,5 +55,5 @@
         <state_interface name="effort"/>
       </joint>
-      <joint name="${prefix}elbow_joint">
+      <joint name="$(arg prefix)elbow_joint">
         <command_interface name="position">
           <param name="min"> ${joint1_PositionMin} </param>
@@ -72,5 +72,5 @@
         <state_interface name="effort"/>
       </joint>
-      <joint name="${prefix}wrist_1_joint">
+      <joint name="$(arg prefix)wrist_1_joint">
         <command_interface name="position">
           <param name="min"> ${joint1_PositionMin} </param>
@@ -89,5 +89,5 @@
         <state_interface name="effort"/>
       </joint>
-      <joint name="${prefix}wrist_2_joint">
+      <joint name="$(arg prefix)wrist_2_joint">
         <command_interface name="position">
           <param name="min"> ${joint1_PositionMin} </param>
@@ -106,5 +106,5 @@
         <state_interface name="effort"/>
       </joint>
-      <joint name="${prefix}wrist_3_joint">
+      <joint name="$(arg prefix)wrist_3_joint">
         <command_interface name="position">
           <param name="min"> ${joint1_PositionMin} </param>

File: urdf/z1.urdf.xacro (robot description, xacro)
@@ -1,8 +1,16 @@
 <?xml version="1.0"?>
 <robot name="z1_description" xmlns:xacro="http://www.ros.org/wiki/xacro">
+    <xacro:arg name="prefix" default="" />
+    <xacro:arg name="simulation_controllers" default="$(find unitree_z1_hw_interface)/config/z1_controllers.yaml" />
+    <xacro:arg name="sim_ignition" default="true" />
+    <xacro:arg name="UnitreeGripper" default="true"/>
     <xacro:include filename="$(find unitree_z1_hw_interface)/urdf/const.xacro"/>
-    <xacro:include filename="$(find unitree_z1_hw_interface)/urdf/gazebo.xacro"/>
-    <xacro:include filename="$(find unitree_z1_hw_interface)/urdf/transmission.xacro"/>
-    <xacro:arg name="UnitreeGripper" default="false"/>
+    <!-- <xacro:include filename="$(find unitree_z1_hw_interface)/urdf/gazebo.xacro"/> -->
+    <!-- <xacro:include filename="$(find unitree_z1_hw_interface)/urdf/transmission.xacro"/> -->
+    <xacro:include filename="$(find unitree_z1_hw_interface)/urdf/z1.ros2_control.xacro"/>
+    <xacro:z1_ros2_control
+    name="z1"
+    prefix="$(arg prefix)"
+    sim_ignition="$(arg sim_ignition)"/>
     <link name="world"/>
     <joint name="base_static_joint" type="fixed">
@@ -33,5 +41,5 @@
         </inertial>
     </link>
-    <joint name="joint1" type="revolute">
+    <joint name="$(arg prefix)shoulder_pan_joint" type="revolute">
         <origin rpy="0 0 0" xyz="0 0 0.0585"/>
         <parent link="link00"/>
@@ -57,5 +65,5 @@
         </inertial>
     </link>
-    <joint name="joint2" type="revolute">
+    <joint name="$(arg prefix)shoulder_lift_joint" type="revolute">
         <origin rpy="0 0 0" xyz="0 0 0.045"/>
         <parent link="link01"/>
@@ -99,5 +107,5 @@
         </inertial>
     </link>
-    <joint name="joint3" type="revolute">
+    <joint name="$(arg prefix)elbow_joint" type="revolute">
         <origin rpy="0 0 0" xyz="-0.35 0 0"/>
         <parent link="link02"/>
@@ -135,5 +143,5 @@
         </inertial>
     </link>
-    <joint name="joint4" type="revolute">
+    <joint name="$(arg prefix)wrist_1_joint" type="revolute">
         <origin rpy="0 0 0" xyz="0.218 0 0.057"/>
         <parent link="link03"/>
@@ -165,5 +173,5 @@
         </inertial>
     </link>
-    <joint name="joint5" type="revolute">
+    <joint name="$(arg prefix)wrist_2_joint" type="revolute">
         <origin rpy="0 0 0" xyz="0.07 0.0 0.0"/>
         <parent link="link04"/>
@@ -189,5 +197,5 @@
         </inertial>
     </link>
-    <joint name="joint6" type="revolute">
+    <joint name="$(arg prefix)wrist_3_joint" type="revolute">
         <origin rpy="0 0 0" xyz="0.0492 0.0 0.0"/>
         <parent link="link05"/>
@@ -273,5 +281,5 @@
             </inertial>
         </link>
-        <xacro:motorTransmission name="Gripper"/>
+        <!--<xacro:motorTransmission name="Gripper"/>-->
         <gazebo reference="gripperStator">
             <self_collide>true</self_collide>
@@ -281,4 +289,5 @@
         </gazebo>
     </xacro:if>
+    <!--
     <xacro:motorTransmission name="1"/>
     <xacro:motorTransmission name="2"/>
@@ -287,3 +296,15 @@
     <xacro:motorTransmission name="5"/>
     <xacro:motorTransmission name="6"/>
+    -->
+    <xacro:if value="$(arg sim_ignition)">
+        Gazebo plugins
+        <gazebo reference="world">
+        </gazebo>
+        <gazebo>
+            <plugin filename = "libign_ros2_control-system.so" name="ign_ros2_contro::IgnitionROS2ControlPlugin">
+                <parameters> $(arg simulation_controllers) </parameters>
+                <controller_manager_node_name> $(arg prefix)controller_manager </controller_manager_node_name>
+            </plugin>
+        </gazebo>
+    </xacro:if>
 </robot>
