Commit message: Fixed state/commands interface export

File: urdf/z1.ros2_control.xacro (robot description, xacro)
@@ -9,4 +9,5 @@
     sim_ignition:=true
     prefix
+    with_gripper:=true
     ">
     <ros2_control name="${name}" type="system">
@@ -17,5 +18,5 @@
         <xacro:unless value="${sim_ignition}">
           <plugin>unitree_z1_hw_interface/UnitreeZ1HWInterface</plugin>
-          <param name="gripper">true</param>
+          <param name="gripper">${with_gripper}</param>
           <!-- add other necessary parameters here -->
         </xacro:unless>
@@ -123,4 +124,23 @@
         <state_interface name="effort"/>
       </joint>
+      <xacro:if value="${with_gripper}">
+          <joint name="$(arg prefix)gripper">
+            <command_interface name="position">
+              <param name="min"> ${Gripper_PositionMin} </param>
+              <param name="max"> ${Gripper_PositionMax} </param>
+            </command_interface>
+            <command_interface name="velocity">
+              <param name="min"> -${velocityMax} </param>
+              <param name="max"> ${velocityMax} </param>
+            </command_interface>
+            <command_interface name="effort">
+              <param name="min"> -${torqueMax} </param>
+              <param name="max"> ${torqueMax} </param>
+            </command_interface>
+            <state_interface name="position"/>
+            <state_interface name="velocity"/>
+            <state_interface name="effort"/>
+          </joint>
+    </xacro:if>
     </ros2_control>
   </xacro:macro>

File: urdf/z1.urdf.xacro (robot description, xacro)
@@ -4,5 +4,5 @@
     <xacro:arg name="simulation_controllers" default="$(find unitree_z1_hw_interface)/config/z1_controllers.yaml" />
     <xacro:arg name="sim_ignition" default="true" />
-    <xacro:arg name="UnitreeGripper" default="true"/>
+    <xacro:arg name="with_gripper" default="true"/>
     <xacro:include filename="$(find unitree_z1_hw_interface)/urdf/const.xacro"/>
     <!-- <xacro:include filename="$(find unitree_z1_hw_interface)/urdf/gazebo.xacro"/> -->
@@ -12,5 +12,6 @@
     name="z1"
     prefix="$(arg prefix)"
-    sim_ignition="$(arg sim_ignition)"/>
+    sim_ignition="$(arg sim_ignition)"
+    with_gripper="$(arg with_gripper)"/>
     <link name="world"/>
     <joint name="base_static_joint" type="fixed">
@@ -227,5 +228,5 @@
         </inertial>
     </link>
-    <xacro:if value="$(arg UnitreeGripper)">
+    <xacro:if value="$(arg with_gripper)">
         <joint name="gripperStator" type="fixed">
             <origin rpy="0 0 0" xyz="0.051 0.0 0.0"/>
