Commit message: Developed hardware interface Tested that state interface is working as expected

File: urdf/z1.urdf.xacro (robot description, xacro)
@@ -254,5 +254,5 @@
             </inertial>
         </link>
-        <joint name="jointGripper" type="revolute">
+        <joint name="gripper" type="revolute">
             <origin rpy="0 0 0" xyz="0.049 0.0 0"/>
             <parent link="gripperStator"/>

Commit message: Testing position and torque control

File: urdf/z1.urdf.xacro (robot description, xacro)
@@ -228,4 +228,10 @@
         </inertial>
     </link>
+    <link name="end_effector"/>
+    <joint name="end_effect_link" type="fixed">
+        <origin rpy="0 0 0" xyz="0.051 0.0 0.0"/>
+        <parent link="link06"/>
+        <child link="end_effector"/>
+    </joint>
     <xacro:if value="$(arg with_gripper)">
         <joint name="gripperStator" type="fixed">
