Commit message: Modified files according to new file structure

File: z1_description/urdf/z1.ros2_control.xacro (robot description, xacro)
@@ -19,5 +19,5 @@
         </xacro:if>
         <xacro:unless value="${sim_ignition}">
-          <plugin>unitree_z1_hw_interface/UnitreeZ1HWInterface</plugin>
+          <plugin>z1_hw_interface/Z1HwInterface</plugin>
           <param name="gripper">${with_gripper}</param>
           <!-- add other necessary parameters here -->

File: z1_description/urdf/z1.urdf.xacro (robot description, xacro)
@@ -3,11 +3,11 @@
     <xacro:arg name="name" default="z1" />
     <xacro:arg name="prefix" default="" />
-    <xacro:arg name="simulation_controllers" default="$(find unitree_z1_hw_interface)/config/z1_controllers.yaml" />
+    <xacro:arg name="simulation_controllers" default="$(find z1_description)/config/z1_controllers.yaml" />
     <xacro:arg name="sim_ignition" default="true" />
     <xacro:arg name="with_gripper" default="true"/>
-    <xacro:include filename="$(find unitree_z1_hw_interface)/urdf/const.xacro"/>
-    <!-- <xacro:include filename="$(find unitree_z1_hw_interface)/urdf/gazebo.xacro"/> -->
-    <!-- <xacro:include filename="$(find unitree_z1_hw_interface)/urdf/transmission.xacro"/> -->
-    <xacro:include filename="$(find unitree_z1_hw_interface)/urdf/z1.ros2_control.xacro"/>
+    <xacro:include filename="$(find z1_description)/urdf/const.xacro"/>
+    <!-- <xacro:include filename="$(find z1_description)/urdf/gazebo.xacro"/> -->
+    <!-- <xacro:include filename="$(find z1_description)/urdf/transmission.xacro"/> -->
+    <xacro:include filename="$(find z1_description)/urdf/z1.ros2_control.xacro"/>
     <xacro:z1_ros2_control
     name="$(arg name)"
@@ -25,5 +25,5 @@
             <origin rpy="0 0 0" xyz="0 0 0"/>
             <geometry>
-                <mesh filename="package://unitree_z1_hw_interface/meshes/visual/z1_Link00.dae" scale="1 1 1"/>
+                <mesh filename="package://z1_description/meshes/visual/z1_Link00.dae" scale="1 1 1"/>
             </geometry>
         </visual>
@@ -55,5 +55,5 @@
             <origin rpy="0 0 0" xyz="0 0 0"/>
             <geometry>
-                <mesh filename="package://unitree_z1_hw_interface/meshes/visual/z1_Link01.dae" scale="1 1 1"/>
+                <mesh filename="package://z1_description/meshes/visual/z1_Link01.dae" scale="1 1 1"/>
             </geometry>
         </visual>
@@ -79,5 +79,5 @@
             <origin rpy="0 0 0" xyz="0 0 0"/>
             <geometry>
-                <mesh filename="package://unitree_z1_hw_interface/meshes/visual/z1_Link02.dae" scale="1 1 1"/>
+                <mesh filename="package://z1_description/meshes/visual/z1_Link02.dae" scale="1 1 1"/>
             </geometry>
         </visual>
@@ -121,5 +121,5 @@
             <origin rpy="0 0 0" xyz="0 0 0"/>
             <geometry>
-                <mesh filename="package://unitree_z1_hw_interface/meshes/visual/z1_Link03.dae" scale="1 1 1"/>
+                <mesh filename="package://z1_description/meshes/visual/z1_Link03.dae" scale="1 1 1"/>
             </geometry>
         </visual>
@@ -157,5 +157,5 @@
             <origin rpy="0 0 0" xyz="0 0 0"/>
             <geometry>
-                <mesh filename="package://unitree_z1_hw_interface/meshes/visual/z1_Link04.dae" scale="1 1 1"/>
+                <mesh filename="package://z1_description/meshes/visual/z1_Link04.dae" scale="1 1 1"/>
             </geometry>
         </visual>
@@ -187,5 +187,5 @@
             <origin rpy="0 0 0" xyz="0 0 0"/>
             <geometry>
-                <mesh filename="package://unitree_z1_hw_interface/meshes/visual/z1_Link05.dae" scale="1 1 1"/>
+                <mesh filename="package://z1_description/meshes/visual/z1_Link05.dae" scale="1 1 1"/>
             </geometry>
         </visual>
@@ -211,5 +211,5 @@
             <origin rpy="0 0 0" xyz="0 0 0"/>
             <geometry>
-                <mesh filename="package://unitree_z1_hw_interface/meshes/visual/z1_Link06.dae" scale="1 1 1"/>
+                <mesh filename="package://z1_description/meshes/visual/z1_Link06.dae" scale="1 1 1"/>
             </geometry>
         </visual>
@@ -244,10 +244,10 @@
             <visual>
                 <geometry>
-                    <mesh filename="package://unitree_z1_hw_interface/meshes/visual/z1_GripperStator.dae" scale="1 1 1"/>
+                    <mesh filename="package://z1_description/meshes/visual/z1_GripperStator.dae" scale="1 1 1"/>
                 </geometry>
             </visual>
             <collision>
                 <geometry>
-                    <mesh filename="package://unitree_z1_hw_interface/meshes/collision/z1_GripperStator.STL" scale="1 1 1"/>
+                    <mesh filename="package://z1_description/meshes/collision/z1_GripperStator.STL" scale="1 1 1"/>
                 </geometry>
             </collision>
@@ -272,10 +272,10 @@
             <visual>
                 <geometry>
-                    <mesh filename="package://unitree_z1_hw_interface/meshes/visual/z1_GripperMover.dae" scale="1 1 1"/>
+                    <mesh filename="package://z1_description/meshes/visual/z1_GripperMover.dae" scale="1 1 1"/>
                 </geometry>
             </visual>
             <collision>
                 <geometry>
-                    <mesh filename="package://unitree_z1_hw_interface/meshes/collision/z1_GripperMover.STL" scale="1 1 1"/>
+                    <mesh filename="package://z1_description/meshes/collision/z1_GripperMover.STL" scale="1 1 1"/>
                 </geometry>
             </collision>
