Commit message: Reformatted and improved URDF files

File: z1_description/urdf/z1.ros2_control.xacro (robot description, xacro)
@@ -5,145 +5,143 @@
 <!-- https://github.com/UniversalRobots/Universal_Robots_ROS2_Description/blob/rolling/urdf/ur.ros2_control.xacro -->
 <robot xmlns:xacro="http://www.ros.org/wiki/xacro">
-  <xacro:macro name="z1_ros2_control" params="
-    name
-    sim_ignition:=true
-    prefix
-    with_gripper:=true
-    ">
-  <!-- <ros2_control name="${name}" type="system"> -->
-    <ros2_control name="${name}" type="system">
-      <hardware>
-        <xacro:if value="${sim_ignition}">
-        <plugin>ign_ros2_control/IgnitionSystem</plugin>
-            <!-- <plugin>gz_ros2_control/GazeboSimSystem</plugin>-->
-        </xacro:if>
-        <xacro:unless value="${sim_ignition}">
-          <plugin>z1_hw_interface/Z1HwInterface</plugin>
-          <param name="gripper">${with_gripper}</param>
-          <!-- add other necessary parameters here -->
-        </xacro:unless>
-      </hardware>
-      <joint name="$(arg prefix)shoulder_pan_joint">
-        <command_interface name="position">
-          <param name="min"> ${joint1_PositionMin} </param>
-          <param name="max"> ${joint1_PositionMax} </param>
-        </command_interface>
-        <command_interface name="velocity">
-          <param name="min"> -${velocityMax} </param>
-          <param name="max"> ${velocityMax} </param>
-        </command_interface>
-        <command_interface name="effort">
-          <param name="min"> -${torqueMax} </param>
-          <param name="max"> ${torqueMax} </param>
-        </command_interface>
-        <state_interface name="position"/>
-        <state_interface name="velocity"/>
-        <state_interface name="effort"/>
-      </joint>
-      <joint name="$(arg prefix)shoulder_lift_joint">
-        <command_interface name="position">
-          <param name="min"> ${joint2_PositionMin} </param>
-          <param name="max"> ${joint2_PositionMax} </param>
-        </command_interface>
-        <command_interface name="velocity">
-          <param name="min"> -${velocityMax} </param>
-          <param name="max"> ${velocityMax} </param>
-        </command_interface>
-        <command_interface name="effort">
-          <param name="min"> -${2*torqueMax} </param>
-          <param name="max"> ${2*torqueMax} </param>
-        </command_interface>
-        <state_interface name="position"/>
-        <state_interface name="velocity"/>
-        <state_interface name="effort"/>
-      </joint>
-      <joint name="$(arg prefix)elbow_joint">
-        <command_interface name="position">
-          <param name="min"> ${joint3_PositionMin} </param>
-          <param name="max"> ${joint3_PositionMax} </param>
-        </command_interface>
-        <command_interface name="velocity">
-          <param name="min"> -${velocityMax} </param>
-          <param name="max"> ${velocityMax} </param>
-        </command_interface>
-        <command_interface name="effort">
-          <param name="min"> -${torqueMax} </param>
-          <param name="max"> ${torqueMax} </param>
-        </command_interface>
-        <state_interface name="position"/>
-        <state_interface name="velocity"/>
-        <state_interface name="effort"/>
-      </joint>
-      <joint name="$(arg prefix)wrist_1_joint">
-        <command_interface name="position">
-          <param name="min"> ${joint4_PositionMin} </param>
-          <param name="max"> ${joint4_PositionMax} </param>
-        </command_interface>
-        <command_interface name="velocity">
-          <param name="min"> -${velocityMax} </param>
-          <param name="max"> ${velocityMax} </param>
-        </command_interface>
-        <command_interface name="effort">
-          <param name="min"> -${torqueMax} </param>
-          <param name="max"> ${torqueMax} </param>
-        </command_interface>
-        <state_interface name="position"/>
-        <state_interface name="velocity"/>
-        <state_interface name="effort"/>
-      </joint>
-      <joint name="$(arg prefix)wrist_2_joint">
-        <command_interface name="position">
-          <param name="min"> ${joint5_PositionMin} </param>
-          <param name="max"> ${joint5_PositionMax} </param>
-        </command_interface>
-        <command_interface name="velocity">
-          <param name="min"> -${velocityMax} </param>
-          <param name="max"> ${velocityMax} </param>
-        </command_interface>
-        <command_interface name="effort">
-          <param name="min"> -${torqueMax} </param>
-          <param name="max"> ${torqueMax} </param>
-        </command_interface>
-        <state_interface name="position"/>
-        <state_interface name="velocity"/>
-        <state_interface name="effort"/>
-      </joint>
-      <joint name="$(arg prefix)wrist_3_joint">
-        <command_interface name="position">
-          <param name="min"> ${joint6_PositionMin} </param>
-          <param name="max"> ${joint6_PositionMax} </param>
-        </command_interface>
-        <command_interface name="velocity">
-          <param name="min"> -${velocityMax} </param>
-          <param name="max"> ${velocityMax} </param>
-        </command_interface>
-        <command_interface name="effort">
-          <param name="min"> -${torqueMax} </param>
-          <param name="max"> ${torqueMax} </param>
-        </command_interface>
-        <state_interface name="position"/>
-        <state_interface name="velocity"/>
-        <state_interface name="effort"/>
-      </joint>
-      <xacro:if value="${with_gripper}">
-          <joint name="$(arg prefix)gripper">
-            <command_interface name="position">
-              <param name="min"> ${Gripper_PositionMin} </param>
-              <param name="max"> ${Gripper_PositionMax} </param>
-            </command_interface>
-            <command_interface name="velocity">
-              <param name="min"> -${velocityMax} </param>
-              <param name="max"> ${velocityMax} </param>
-            </command_interface>
-            <command_interface name="effort">
-              <param name="min"> -${torqueMax} </param>
-              <param name="max"> ${torqueMax} </param>
-            </command_interface>
-            <state_interface name="position"/>
-            <state_interface name="velocity"/>
-            <state_interface name="effort"/>
-          </joint>
-    </xacro:if>
-    </ros2_control>
-  </xacro:macro>
+    <xacro:macro name="z1_ros2_control" params="
+        name:='z1'
+        sim_ignition:=true
+        prefix:=''
+        with_gripper:=true
+        ">
+        <ros2_control name="${name}" type="system">
+            <hardware>
+                <xacro:if value="${sim_ignition}">
+                    <plugin>ign_ros2_control/IgnitionSystem</plugin>
+                </xacro:if>
+                <xacro:unless value="${sim_ignition}">
+                    <plugin>z1_hw_interface/Z1HwInterface</plugin>
+                    <param name="gripper">${with_gripper}</param>
+                    <!-- add other necessary parameters here -->
+                </xacro:unless>
+            </hardware>
+            <joint name="joint1">
+                <command_interface name="position">
+                    <param name="min"> ${joint1_PositionMin} </param>
+                    <param name="max"> ${joint1_PositionMax} </param>
+                </command_interface>
+                <command_interface name="velocity">
+                    <param name="min"> -${velocityMax} </param>
+                    <param name="max"> ${velocityMax} </param>
+                </command_interface>
+                <command_interface name="effort">
+                    <param name="min"> -${torqueMax} </param>
+                    <param name="max"> ${torqueMax} </param>
+                </command_interface>
+                <state_interface name="position"/>
+                <state_interface name="velocity"/>
+                <state_interface name="effort"/>
+            </joint>
+            <joint name="joint2">
+                <command_interface name="position">
+                    <param name="min"> ${joint2_PositionMin} </param>
+                    <param name="max"> ${joint2_PositionMax} </param>
+                </command_interface>
+                <command_interface name="velocity">
+                    <param name="min"> -${velocityMax} </param>
+                    <param name="max"> ${velocityMax} </param>
+                </command_interface>
+                <command_interface name="effort">
+                    <param name="min"> -${torqueMax} </param>
+                    <param name="max"> ${torqueMax} </param>
+                </command_interface>
+                <state_interface name="position"/>
+                <state_interface name="velocity"/>
+                <state_interface name="effort"/>
+            </joint>
+            <joint name="joint3">
+                <command_interface name="position">
+                    <param name="min"> ${joint3_PositionMin} </param>
+                    <param name="max"> ${joint3_PositionMax} </param>
+                </command_interface>
+                <command_interface name="velocity">
+                    <param name="min"> -${velocityMax} </param>
+                    <param name="max"> ${velocityMax} </param>
+                </command_interface>
+                <command_interface name="effort">
+                    <param name="min"> -${torqueMax} </param>
+                    <param name="max"> ${torqueMax} </param>
+                </command_interface>
+                <state_interface name="position"/>
+                <state_interface name="velocity"/>
+                <state_interface name="effort"/>
+            </joint>
+            <joint name="joint4">
+                <command_interface name="position">
+                    <param name="min"> ${joint4_PositionMin} </param>
+                    <param name="max"> ${joint4_PositionMax} </param>
+                </command_interface>
+                <command_interface name="velocity">
+                    <param name="min"> -${velocityMax} </param>
+                    <param name="max"> ${velocityMax} </param>
+                </command_interface>
+                <command_interface name="effort">
+                    <param name="min"> -${torqueMax} </param>
+                    <param name="max"> ${torqueMax} </param>
+                </command_interface>
+                <state_interface name="position"/>
+                <state_interface name="velocity"/>
+                <state_interface name="effort"/>
+            </joint>
+            <joint name="joint5">
+                <command_interface name="position">
+                    <param name="min"> ${joint5_PositionMin} </param>
+                    <param name="max"> ${joint5_PositionMax} </param>
+                </command_interface>
+                <command_interface name="velocity">
+                    <param name="min"> -${velocityMax} </param>
+                    <param name="max"> ${velocityMax} </param>
+                </command_interface>
+                <command_interface name="effort">
+                    <param name="min"> -${torqueMax} </param>
+                    <param name="max"> ${torqueMax} </param>
+                </command_interface>
+                <state_interface name="position"/>
+                <state_interface name="velocity"/>
+                <state_interface name="effort"/>
+            </joint>
+            <joint name="joint6">
+                <command_interface name="position">
+                    <param name="min"> ${joint6_PositionMin} </param>
+                    <param name="max"> ${joint6_PositionMax} </param>
+                </command_interface>
+                <command_interface name="velocity">
+                    <param name="min"> -${velocityMax} </param>
+                    <param name="max"> ${velocityMax} </param>
+                </command_interface>
+                <command_interface name="effort">
+                    <param name="min"> -${torqueMax} </param>
+                    <param name="max"> ${torqueMax} </param>
+                </command_interface>
+                <state_interface name="position"/>
+                <state_interface name="velocity"/>
+                <state_interface name="effort"/>
+            </joint>
+            <xacro:if value="${with_gripper}">
+                <joint name="jointGripper">
+                    <command_interface name="position">
+                        <param name="min"> ${Gripper_PositionMin} </param>
+                        <param name="max"> ${Gripper_PositionMax} </param>
+                    </command_interface>
+                    <command_interface name="velocity">
+                        <param name="min"> -${velocityMax} </param>
+                        <param name="max"> ${velocityMax} </param>
+                    </command_interface>
+                    <command_interface name="effort">
+                        <param name="min"> -${torqueMax} </param>
+                        <param name="max"> ${torqueMax} </param>
+                    </command_interface>
+                    <state_interface name="position"/>
+                    <state_interface name="velocity"/>
+                    <state_interface name="effort"/>
+                </joint>
+            </xacro:if>
+        </ros2_control>
+    </xacro:macro>
 </robot>

File: z1_description/urdf/z1.urdf.xacro (robot description, xacro)
@@ -7,12 +7,7 @@
     <xacro:arg name="with_gripper" default="true"/>
     <xacro:include filename="$(find z1_description)/urdf/const.xacro"/>
-    <!-- <xacro:include filename="$(find z1_description)/urdf/gazebo.xacro"/> -->
-    <!-- <xacro:include filename="$(find z1_description)/urdf/transmission.xacro"/> -->
+    <xacro:include filename="$(find z1_description)/urdf/gazebo.xacro"/>
     <xacro:include filename="$(find z1_description)/urdf/z1.ros2_control.xacro"/>
-    <xacro:z1_ros2_control
-    name="$(arg name)"
-    prefix="$(arg prefix)"
-    sim_ignition="$(arg sim_ignition)"
-    with_gripper="$(arg with_gripper)"/>
+    <xacro:include filename="$(find z1_description)/urdf/transmission.xacro"/>
     <link name="world"/>
     <joint name="base_static_joint" type="fixed">
@@ -43,5 +38,5 @@
         </inertial>
     </link>
-    <joint name="$(arg prefix)shoulder_pan_joint" type="revolute">
+    <joint name="joint1" type="revolute">
         <origin rpy="0 0 0" xyz="0 0 0.0585"/>
         <parent link="link00"/>
@@ -67,5 +62,5 @@
         </inertial>
     </link>
-    <joint name="$(arg prefix)shoulder_lift_joint" type="revolute">
+    <joint name="joint2" type="revolute">
         <origin rpy="0 0 0" xyz="0 0 0.045"/>
         <parent link="link01"/>
@@ -109,5 +104,5 @@
         </inertial>
     </link>
-    <joint name="$(arg prefix)elbow_joint" type="revolute">
+    <joint name="joint3" type="revolute">
         <origin rpy="0 0 0" xyz="-0.35 0 0"/>
         <parent link="link02"/>
@@ -145,5 +140,5 @@
         </inertial>
     </link>
-    <joint name="$(arg prefix)wrist_1_joint" type="revolute">
+    <joint name="joint4" type="revolute">
         <origin rpy="0 0 0" xyz="0.218 0 0.057"/>
         <parent link="link03"/>
@@ -175,5 +170,5 @@
         </inertial>
     </link>
-    <joint name="$(arg prefix)wrist_2_joint" type="revolute">
+    <joint name="joint5" type="revolute">
         <origin rpy="0 0 0" xyz="0.07 0.0 0.0"/>
         <parent link="link04"/>
@@ -199,5 +194,5 @@
         </inertial>
     </link>
-    <joint name="$(arg prefix)wrist_3_joint" type="revolute">
+    <joint name="joint6" type="revolute">
         <origin rpy="0 0 0" xyz="0.0492 0.0 0.0"/>
         <parent link="link05"/>
@@ -229,12 +224,6 @@
         </inertial>
     </link>
-    <link name="end_effector"/>
-    <joint name="end_effect_link" type="fixed">
-        <origin rpy="0 0 0" xyz="0.051 0.0 0.0"/>
-        <parent link="link06"/>
-        <child link="end_effector"/>
-    </joint>
     <xacro:if value="$(arg with_gripper)">
-        <joint name="gripperStator" type="fixed">
+        <joint name="gripperStatorLink" type="fixed">
             <origin rpy="0 0 0" xyz="0.051 0.0 0.0"/>
             <parent link="link06"/>
@@ -261,5 +250,5 @@
             </inertial>
         </link>
-        <joint name="gripper" type="revolute">
+        <joint name="jointGripper" type="revolute">
             <origin rpy="0 0 0" xyz="0.049 0.0 0"/>
             <parent link="gripperStator"/>
@@ -289,5 +278,4 @@
             </inertial>
         </link>
-        <!--<xacro:motorTransmission name="Gripper"/>-->
         <gazebo reference="gripperStator">
             <self_collide>true</self_collide>
@@ -297,19 +285,7 @@
         </gazebo>
     </xacro:if>
-    <!--
-    <xacro:motorTransmission name="1"/>
-    <xacro:motorTransmission name="2"/>
-    <xacro:motorTransmission name="3"/>
-    <xacro:motorTransmission name="4"/>
-    <xacro:motorTransmission name="5"/>
-    <xacro:motorTransmission name="6"/>
-    -->
     <xacro:if value="$(arg sim_ignition)">
-        Gazebo plugins
-        <gazebo reference="world">
-        </gazebo>
+        <gazebo reference="world"/>
         <gazebo>
-        <!-- <plugin filename = "libign_ros2_control-system.so" name="ign_ros2_control::IgnitionROS2ControlPlugin">-->
-        <!-- <plugin filename="ign_ros2_control-system" name="ign_ros2_control::IgnitionROS2ControlPlugin"> -->
             <plugin filename="libign_ros2_control-system.so" name="ign_ros2_control::IgnitionROS2ControlPlugin">
                 <parameters> $(arg simulation_controllers) </parameters>
@@ -320,3 +296,8 @@
         </gazebo>
     </xacro:if>
+    <xacro:z1_ros2_control
+        name="$(arg name)"
+        prefix="$(arg prefix)"
+        sim_ignition="$(arg sim_ignition)"
+        with_gripper="$(arg with_gripper)"/>
 </robot>
