Commit message: added initial configuration for gazebo simulation in z1.ros2_control.xacro

File: z1_description/urdf/z1.ros2_control.xacro (robot description, xacro)
@@ -3,7 +3,9 @@
 <!-- their robots, but with data ported for the Z1 manipulator from alientree.       -->
 <!-- Source to the original file:                                                    -->
-<!-- https://github.com/UniversalRobots/Universal_Robots_ROS2_Description/blob/rolling/urdf/ur.ros2_control.xacro -->
+<!--
+https://github.com/UniversalRobots/Universal_Robots_ROS2_Description/blob/rolling/urdf/ur.ros2_control.xacro -->
 <robot xmlns:xacro="http://www.ros.org/wiki/xacro">
-    <xacro:macro name="z1_ros2_control" params="
+    <xacro:macro name="z1_ros2_control"
+        params="
         name:='z1'
         sim_ignition:=true
@@ -13,4 +15,7 @@
         <ros2_control name="${name}" type="system">
             <hardware>
+                <!-- <xacro:if value="${coppelia}">
+                    <plugin>z1_coppelia_hw/Z1EffortFakeHardware</plugin>
+                </xacro:if> -->
                 <xacro:if value="${sim_ignition}">
                     <plugin>ign_ros2_control/IgnitionSystem</plugin>
@@ -19,5 +24,4 @@
                     <plugin>z1_hw_interface/Z1HwInterface</plugin>
                     <param name="gripper">${with_gripper}</param>
-                    <!-- add other necessary parameters here -->
                 </xacro:unless>
             </hardware>
@@ -31,7 +35,7 @@
                     <param name="max"> ${torqueMax} </param>
                 </command_interface>
-                <state_interface name="position"/>
-                <state_interface name="velocity"/>
-                <state_interface name="effort"/>
+                <state_interface name="position" />
+                <state_interface name="velocity" />
+                <state_interface name="effort" />
             </joint>
             <joint name="joint2">
@@ -40,11 +44,20 @@
                     <param name="max"> ${joint2_PositionMax} </param>
                 </command_interface>
-                <command_interface name="effort">
+                <command_interface
+                    name="effort">
                     <param name="min"> -${torqueMax} </param>
                     <param name="max"> ${torqueMax} </param>
                 </command_interface>
-                <state_interface name="position"/>
-                <state_interface name="velocity"/>
-                <state_interface name="effort"/>
+                <xacro:if value="${sim_ignition}">
+                    <!-- setting initial position in gazebo -->
+                    <state_interface name="position">
+                        <param name="initial_value">1.57</param>
+                    </state_interface>
+                </xacro:if>
+                <xacro:unless value="${sim_ignition}">
+                    <state_interface name="position" />
+                </xacro:unless>
+                <state_interface name="velocity" />
+                <state_interface name="effort" />
             </joint>
             <joint name="joint3">
@@ -57,7 +70,15 @@
                     <param name="max"> ${torqueMax} </param>
                 </command_interface>
-                <state_interface name="position"/>
-                <state_interface name="velocity"/>
-                <state_interface name="effort"/>
+                <xacro:if value="${sim_ignition}">
+                    <!-- setting initial position in gazebo -->
+                    <state_interface name="position">
+                        <param name="initial_value">-1.57</param>
+                    </state_interface>
+                </xacro:if>
+                <xacro:unless value="${sim_ignition}">
+                    <state_interface name="position" />
+                </xacro:unless>
+                <state_interface name="velocity" />
+                <state_interface name="effort" />
             </joint>
             <joint name="joint4">
@@ -70,7 +91,7 @@
                     <param name="max"> ${torqueMax} </param>
                 </command_interface>
-                <state_interface name="position"/>
-                <state_interface name="velocity"/>
-                <state_interface name="effort"/>
+                <state_interface name="position" />
+                <state_interface name="velocity" />
+                <state_interface name="effort" />
             </joint>
             <joint name="joint5">
@@ -83,7 +104,7 @@
                     <param name="max"> ${torqueMax} </param>
                 </command_interface>
-                <state_interface name="position"/>
-                <state_interface name="velocity"/>
-                <state_interface name="effort"/>
+                <state_interface name="position" />
+                <state_interface name="velocity" />
+                <state_interface name="effort" />
             </joint>
             <joint name="joint6">
@@ -96,7 +117,7 @@
                     <param name="max"> ${torqueMax} </param>
                 </command_interface>
-                <state_interface name="position"/>
-                <state_interface name="velocity"/>
-                <state_interface name="effort"/>
+                <state_interface name="position" />
+                <state_interface name="velocity" />
+                <state_interface name="effort" />
             </joint>
             <xacro:if value="${with_gripper}">
@@ -110,7 +131,7 @@
                         <param name="max"> ${torqueMax} </param>
                     </command_interface>
-                    <state_interface name="position"/>
-                    <state_interface name="velocity"/>
-                    <state_interface name="effort"/>
+                    <state_interface name="position" />
+                    <state_interface name="velocity" />
+                    <state_interface name="effort" />
                 </joint>
             </xacro:if>
